File: Robocik-Plytka_uniwersalna_silnikiDC/Robocik-Plytka_uniwersalna_silnikiDC.sch (KiCad schematic (older format))
At the start: 50 parts, among them IC1 ACSL-6400-00TE, IC2 ACSL-6400-00TE, IC3 L6205D, Q1 Q_NPN_BCE, Q2 Q_NPN_BCE, Q3 Q_NPN_BCE, Q4 Q_NPN_BCE, Q5 Q_NPN_BCE, Q6 Q_NPN_BCE, U1 STM32F103C8Tx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

Commit message: Added tantalum capacitors on the output of linear regulators, removed second photocoupler and simplified flags. Removed jumpers. Fixed RC filters on ENABLE pins.
Parts:
- removed IC2: ACSL-6400-00TE, SOIC127P599X173-16N, symbol ACSL-6400-00TE:ACSL-6400-00TE
- removed J?: ENGB, symbol Connector_Generic:Conn_01x02
- removed JP1, JP2, JP3, JP4, JP5: Jumper_2_Bridged, symbol Jumper:Jumper_2_Bridged
- removed Q4, Q5, Q6: Q_NPN_BCE, symbol Device:Q_NPN_BCE
- removed R12, R13, R14, R3, R4, R7, R8: 4k7, symbol Device:R_Small
- added C11, C12: 47uF, symbol Device:CP_Small
- J2: renamed from J?; value ENGA -> ENG
- gave numbers to parts that had none: 2
Connections:
- net labels added: EN, ENG1, ENG2, IN1, IN2
- net labels removed: ENA, ENB, ENGA1, ENGA2, ENGB1, ENGB2, IN1A, IN1B, IN2A, IN2B
- wire segments 93 -> 72
Other:
- note added: "13.02.2020"
- note added: "DC motor driver, photocoupler and MCU PCB"
- note added: "Igor Zieliński\nWiktor Paluch"
- moved on the sheet: C1, C10, C2, C3, C4, C5, C6, C7, C8, C9, D1, D2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
